File: PCB_Project/electrophy_2/electrophy_2.kicad_pcb (KiCad board)
At the start: 4 copper layers, 35 x 35 mm, 47 parts, among them IC1 ESP32-C3FN4, J1 USB_C_Receptacle_USB2.0_14P, J3 Conn_01x04, U1 LSM6DSV320XTR, U2 BQ21040DBV, U3 TPS27081ADDCR, U4 USBLC6-2SC6, U5 MIC5504-3.3YM5, Y1 40MHZ 15pf, Y2 32 KHz

Commit message: changed Iset resistor value in schematic
Parts:
- R9: value 26k -> 10k-26k
Changed lines of the file:
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@@
 			)
 		)
-		(property "Value" "26k"
+		(property "Value" "10k-26k"
 			(at 0 1.17 90)
 			(layer "F.Fab")
