File: PCB_Project/electrophy_2/electrophy_2.kicad_sch (KiCad schematic)
At the start: 45 parts, among them IC1 ESP32-C3FN4, J1 USB_C_Receptacle_USB2.0_14P, J3 Conn_01x04, SW2 SW_Push, U1 LSM6DSV320XTR, U2 BQ21040DBV, U3 TPS27081ADDCR, U4 USBLC6-2SC6, U5 MIC5504-3.3YM5, Y1 40MHZ 15pf, Y2 32 KHz

Commit message: PCB draft
Parts:
- J3: footprint Connector_FFC-FPC:Amphenol_F32R-1A7x1-11004_1x04-1MP_P0.5mm_Horizontal -> pogo_pads_4:pogo_pads_4
Connections:
- net BAT_V: now also C2.1, R3.1, U3.2 (VOUT), U3.3 (VOUT), U5.1 (VIN); no longer BAT1.1 (Pin_1), R11.1, R13.1, SW2.1, U2.2 (OUT), U3.4 (VIN)
- net SCL: now also J3.3 (Pin_3); no longer J3.4 (Pin_4)
- net SDA: now also J3.4 (Pin_4); no longer J3.3 (Pin_3)
- new net: BAT1.1 (Pin_1), R11.1, R13.1, SW2.1, U2.2 (OUT), U3.4 (VIN)
Changed lines of the file:
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@@
 	)
 	(junction
-		(at 90.17 30.48)
-		(diameter 0)
-		(color 0 0 0 0)
-	)
-	(junction
 		(at 234.95 38.1)
 		(diameter 0)
@@
 	(wire
 		(pts
-			(xy 45.72 124.46) (xy 54.61 124.46)
-		)
-		(stroke
-			(width 0)
-			(type default)
-		)
-	)
-	(wire
-		(pts
 			(xy -71.12 43.18) (xy -71.12 44.45)
 		)
@@
 	(wire
 		(pts
-			(xy 83.82 30.48) (xy 90.17 30.48)
+			(xy 83.82 30.48) (xy 99.06 30.48)
 		)
 		(stroke
@@
 	(wire
 		(pts
+			(xy 46.99 121.92) (xy 54.61 121.92)
+		)
+		(stroke
+			(width 0)
+			(type default)
+		)
+	)
+	(wire
+		(pts
 			(xy 220.98 44.45) (xy 231.14 44.45)
 		)
@@
 	(wire
 		(pts
+			(xy 144.78 21.59) (xy 144.78 30.48)
+		)
+		(stroke
+			(width 0)
+			(type default)
+		)
+	)
+	(wire
+		(pts
 			(xy 213.36 124.46) (xy 199.39 124.46)
 		)
@@
 	(wire
 		(pts
-			(xy 59.69 31.75) (xy 48.26 31.75)
+			(xy 46.99 124.46) (xy 54.61 124.46)
 		)
 		(stroke
@@
 	(wire
 		(pts
-			(xy 129.54 30.48) (xy 140.97 30.48)
+			(xy 59.69 31.75) (xy 48.26 31.75)
 		)
 		(stroke
@@
 	(wire
 		(pts
-			(xy 179.07 158.75) (xy 179.07 160.02)
+			(xy 129.54 30.48) (xy 140.97 30.48)
 		)
 		(stroke
@@
 	(wire
 		(pts
-			(xy 250.19 153.67) (xy 241.3 153.67)
+			(xy 179.07 158.75) (xy 179.07 160.02)
 		)
 		(stroke
@@
 	(wire
 		(pts
-			(xy 45.72 121.92) (xy 54.61 121.92)
+			(xy 250.19 153.67) (xy 241.3 153.67)
 		)
 		(stroke
@@
 	(wire
 		(pts
-			(xy 90.17 30.48) (xy 99.06 30.48)
-		)
-		(stroke
-			(width 0)
-			(type default)
-		)
-	)
-	(wire
-		(pts
 			(xy 116.84 53.34) (xy 116.84 52.07)
 		)
@@
 	(wire
 		(pts
-			(xy 90.17 17.78) (xy 90.17 30.48)
-		)
-		(stroke
-			(width 0)
-			(type default)
-		)
-	)
-	(wire
-		(pts
 			(xy 199.39 153.67) (xy 199.39 147.32)
 		)
@@
 	(wire
 		(pts
-			(xy 87.63 17.78) (xy 90.17 17.78)
-		)
-		(stroke
-			(width 0)
-			(type default)
-		)
-	)
-	(wire
-		(pts
 			(xy 238.76 44.45) (xy 248.92 44.45)
 		)
@@
 	(global_label "BAT_V"
 		(shape input)
-		(at 87.63 17.78 180)
+		(at 144.78 21.59 180)
 		(fields_autoplaced yes)
 		(effects
@@
 		)
 		(property "Intersheetrefs" "${INTERSHEET_REFS}"
-			(at 79.2624 17.78 0)
+			(at 136.4124 21.59 0)
 			(hide yes)
 			(show_name no)
@@
 	(global_label "SCL"
 		(shape input)
-		(at 45.72 124.46 180)
+		(at 46.99 121.92 180)
 		(fields_autoplaced yes)
 		(effects
@@
 		)
 		(property "Intersheetrefs" "${INTERSHEET_REFS}"
-			(at 39.2272 124.46 0)
+			(at 40.4972 121.92 0)
 			(hide yes)
 			(show_name no)
@@
 	(global_label "SDA"
 		(shape input)
-		(at 45.72 121.92 180)
+		(at 46.99 124.46 180)
 		(fields_autoplaced yes)
 		(effects
@@
 		)
 		(property "Intersheetrefs" "${INTERSHEET_REFS}"
-			(at 39.1667 121.92 0)
+			(at 40.4367 124.46 0)
 			(hide yes)
 			(show_name no)
@@
 			)
 		)
-		(property "Footprint" "Connector_FFC-FPC:Amphenol_F32R-1A7x1-11004_1x04-1MP_P0.5mm_Horizontal"
+		(property "Footprint" "pogo_pads_4:pogo_pads_4"
 			(at 59.69 119.38 0)
 			(hide yes)

Commit message: added CC1 and CC2 resistors
Parts:
- added R16, R17: 5.1k, Resistor_SMD:R_0402_1005Metric_Pad0.72x0.64mm_HandSolder, symbol Device:R_Small_US
- renumbered STA2 to CH1, SW2 to ON1, STA1 to S1
Connections:
- net GND: now also R16.2, R17.2
- net at J1.A5 (CC1): now also R16.1
- net at J1.B5 (CC2): now also R17.1
Other:
- moved on the sheet: BAT1, C1, C10, C2, C3, CH1, H1, H2, H3, J1, J3, ON1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

Commit message: re-uploaded this version because of DFM issue
Parts:
- R3: value 1k -> 10k
Changed lines of the file:
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@@
 			)
 		)
-		(property "Value" "1k"
+		(property "Value" "10k"
 			(at 143.51 34.29 0)
 			(show_name no)

Commit message: changed Iset resistor value in schematic
Parts:
- R9: value 26k -> 10k-26k
Changed lines of the file:
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@@
 			)
 		)
-		(property "Value" "26k"
+		(property "Value" "10k-26k"
 			(at 24.13 39.37 0)
 			(show_name no)
